Commit message: modified:   .vscode/settings.json 	modified:   src/racecar_description/urdf/sensors/camera.xacro 	modified:   src/racecar_gazebo/config/move_base_config/base_local_planner_params.yaml 	modified:   src/racecar_gazebo/config/move_base_config/costmap_common_params.yaml 	modified:   src/racecar_gazebo/config/move_base_config/global_costmap_params.yaml 	modified:   src/racecar_gazebo/config/move_base_config/local_costmap_params.yaml 	modified:   src/racecar_gazebo/launch/move_base_nav.launch 	modified:   src/racecar_gazebo/scripts/odometry.py

File: src/racecar_description/urdf/sensors/camera.xacro (robot description, xacro)
@@ -13,5 +13,5 @@
 		<origin xyz=" 0 0 0 " rpy="1.57 0 1.57" />
 		<geometry>
-		    <mesh filename="package://racecar_description/meshes/S1030-0315.dae" scale="0.1 0.1 0.1" />
+		    <box size="0.05 0.05 0.05" />
 		</geometry>
 	    </visual>
