Commit message: modified:   src/racecar_description/urdf/racecar.urdf.xacro 	deleted:    src/racecar_gazebo/launch/integrated_navigation.launch 	modified:   src/racecar_gazebo/launch/point_navigation.launch 	deleted:    src/racecar_gazebo/launch/racecar_gazebo.launch 	modified:   src/racecar_gazebo/scripts/point_navigation.py 	deleted:    src/racecar_gazebo/scripts/velocity_mixer.py

File: src/racecar_description/urdf/racecar.urdf.xacro (robot description, xacro)
@@ -83,13 +83,4 @@
     </inertial>
   </xacro:macro>
-  <link name="imu_link">
-    <inertial>
-      <origin xyz="0 0 0"/>
-      <mass value="0.01"/>
-      <inertia ixx="1e-5" ixy="0" ixz="0"
-              iyy="1e-5" iyz="0"
-              izz="1e-5"/>
-    </inertial>
-  </link>
   <xacro:macro name="battery" params="prefix reflect">
     <joint name="chassis_to_${prefix}_battery" type="fixed">

Commit message: modified:   .vscode/settings.json 	modified:   src/racecar_description/urdf/racecar.urdf.xacro 	modified:   src/racecar_gazebo/config/racecar_control.yaml 	new file:   src/racecar_gazebo/launch/auto_run.launch 	modified:   src/racecar_gazebo/scripts/drive_controller.py 	new file:   src/racecar_gazebo/scripts/obstacle_avoidance.py

File: src/racecar_description/urdf/racecar.urdf.xacro (robot description, xacro)
@@ -32,5 +32,5 @@
   <xacro:property name="axle_eff_limit" value="5.12766"/>
   <xacro:property name="axle_vel_limit" value="244.8696"/>
-  <xacro:property name="servo_stall_torque" value="0.5649"/>
+  <xacro:property name="servo_stall_torque" value="10.0"/>
   <xacro:property name="servo_no_load_speed" value="4.553"/>
   <xacro:property name="layer_mass"   value="0.0" />
@@ -202,5 +202,7 @@
                  child="${lr_prefix}_steering_link"/>
     <link name="${lr_prefix}_steering_link">
-      <xacro:null_inertial/>
+      <inertial>
+        <mass value="0.1"/> <inertia ixx="0.01" ixy="0" ixz="0" iyy="0.01" iyz="0" izz="0.01"/>
+      </inertial>
     </link>
     <joint name="${lr_prefix}_steering_joint" type="revolute">
@@ -210,4 +212,5 @@
       <limit lower="${-degrees_45}" upper="${degrees_45}"
              effort="${servo_stall_torque}" velocity="${servo_no_load_speed}"/>
+      <dynamics damping = "1.0" friction = "0.5"/>
     </joint>
     <transmission name="${lr_prefix}_steering_trans">
